Commit message: Initial chromeo example

File: examples/pybullet/construction/framefab_kr6_r900_support/urdf/kr6_r900_workspace.urdf (robot description, URDF)
Before this commit: robot kr6_r900_workspace, 16 links, 15 joints
Links:
- link eef_base_link: geometry collision mesh filename=../../asw_end_effector/meshes/collision/asw_hotend_end_effe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 scale=.001 .001 .001; visual mesh filename=../../asw_end_effector/meshes/visual/asw_hotend_end_effecto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 scale=.001 .001 .001
- link material_feeder_material_feeder: geometry collision mesh filename=../../asw_material_feeder/meshes/collision/asw_material_fee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 scale=.001 .001 .001; visual mesh filename=../../asw_material_feeder/meshes/visual/asw_material_feeder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 scale=.001 .001 .001
- link robot_base_link: geometry collision mesh filename=../../kuka_kr6_support/meshes/kr6_agilus/collision/base_lin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; visual mesh filename=../../kuka_kr6_support/meshes/kr6_agilus/visual/base_link.d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
- link robot_link_1: geometry collision mesh filename=../../kuka_kr6_support/meshes/kr6_agilus/collision/link_1.s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; visual mesh filename=../../kuka_kr6_support/meshes/kr6_agilus/visual/link_1.dae
- link robot_link_2: geometry collision mesh filename=../../kuka_kr6_support/meshes/kr6r900sixx/collision/link_2.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; visual mesh filename=../../kuka_kr6_support/meshes/kr6r900sixx/visual/link_2.dae
- link robot_link_3: geometry collision mesh filename=../../kuka_kr6_support/meshes/kr6_agilus/collision/link_3.s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; visual mesh filename=../../kuka_kr6_support/meshes/kr6_agilus/visual/link_3.dae
- link robot_link_4: geometry collision mesh filename=../../kuka_kr6_support/meshes/kr6r900sixx/collision/link_4.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; visual mesh filename=../../kuka_kr6_support/meshes/kr6r900sixx/visual/link_4.dae
- link robot_link_5: geometry collision mesh filename=../../kuka_kr6_support/meshes/kr6_agilus/collision/link_5.s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; visual mesh filename=../../kuka_kr6_support/meshes/kr6_agilus/visual/link_5.dae
- link robot_link_6: geometry collision mesh filename=../../kuka_kr6_support/meshes/kr6_agilus/collision/link_6.s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; visual mesh filename=../../kuka_kr6_support/meshes/kr6_agilus/visual/link_6.dae
- link workspace_objects: geometry collision mesh filename=../../framefab_kr6_r900_support/meshes/collision/MIT_3-412_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; visual mesh filename=../../framefab_kr6_r900_support/meshes/visual/MIT_3-412_wor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
