Commit message: Construction progress

File: examples/pybullet/construction/framefab_kr6_r900_support/urdf/kr6_r900.urdf (robot description, URDF)
Before this commit: robot kr6_r900_workspace, 16 links, 15 joints
Links:
- removed link base_link
- removed link material_feeder_material_feeder
- removed link material_feeder_mount_point
- removed link workspace_base_link
- removed link workspace_objects
Joints:
- removed joint link_3_to_link_3_mount_point
- removed joint mount_point_to_material_feeder
- removed joint workspace_baselink_to_objects
- removed joint world_to_base
- removed joint world_to_workspace

Commit message: Modified kr6 joint limits

File: examples/pybullet/construction/framefab_kr6_r900_support/urdf/kr6_r900.urdf (robot description, URDF)
Before this commit: robot kr6_r900_workspace, 11 links, 10 joints
Joints:
- joint robot_joint_a1: limit lower=-2.96705972839 upper=2.96705972839 effort=0 velocity=6.28318530718 -> lower=-1.57 upper=1.57 effort=0 velocity=6.28318530718
- joint robot_joint_a6: limit lower=-6.10865238198 upper=6.10865238198 effort=0 velocity=10.7337748998 -> lower=-3.14159 upper=3.14159 effort=0 velocity=10.7337748998
