Commit message: Removing environment from urdf

File: examples/pybullet/construction/framefab_kr6_r900_support/urdf/kr6_r900_mit_suction_gripper.urdf (robot description, URDF)
Before this commit: robot kr6_r900_mit_suction_gripper, 14 links, 13 joints
Links:
- removed link workspace_objects
Joints:
- removed joint workspace_baselink_to_objects
